Commit message: Switch robot_v2 sim model to claude_description (ros2_control)
Reemplaza el modelo robot_v2 por la version de claude_description que usa
ros2_control + diff_drive_controller (en vez de libgazebo_ros_diff_drive):

- body.xacro: nuevo export (anade bola_v1_1/sim_caster_v8, conserva bloque
  <ros2_control>); root->body_link, meshes->package://test_bot.
- robot_v2.gazebo: plugin gazebo_ros2_control + camara + imu + friccion.
- config/controllers.yaml: diff_drive_controller + joint_state_broadcaster
  (sep 0.169 m, radio 0.0325 m).
- launch_sim.launch.py: spawnea joint_state_broadcaster y diff_drive_controller
  tras spawn_entity (event handlers).
- README: notas ros2_control, deps (gazebo-ros2-control) y tuning.

Co-Authored-By: Claude Opus 4.8 <noreply@anthropic.com>

File: description/robot_v2/body.xacro (robot description, xacro)
@@ -1,9 +1,11 @@
 <?xml version="1.0" ?>
-<robot name="robot_v2_urdf" xmlns:xacro="http://www.ros.org/wiki/xacro">
-<!-- Fragmento de cuerpo del robot_v2 (export Fusion360), adaptado para test_bot:
+<robot name="robot_v2_urdf_v2" xmlns:xacro="http://www.ros.org/wiki/xacro">
+<!-- Fragmento de cuerpo del robot_v2_urdf_v2 (export Fusion360, version con
+     ros2_control), adaptado para test_bot:
      - root 'base_link' renombrado a 'body_link' (el wrapper aporta base_link/base_footprint).
-     - rutas de mesh apuntan a package://test_bot/description/meshes.
-     - joints de rueda 'Revolute 17/18' renombrados a right/left_wheel_joint.
-     - SIN includes de materials/trans/gazebo (los aporta robot_v2.urdf.xacro). -->
+     - rutas de mesh -> package://test_bot/description/meshes.
+     - joints de rueda ya vienen como left/right_wheel_joint.
+     - se conserva el bloque <ros2_control> (interfaces de hardware Gazebo).
+     - SIN includes de materials/gazebo (los aporta robot_v2.urdf.xacro / robot_v2.gazebo). -->
 <link name="body_link">
   <inertial>
@@ -326,8 +328,8 @@
   </collision>
 </link>
-<link name="sim_caster_v7_1">
-  <inertial>
-    <origin xyz="-0.011649938340071692 -0.011649938044252545 -0.003324314430276934" rpy="0 0 0"/>
-    <mass value="0.00517152232374024"/>
+<link name="sim_caster_v8_1">
+  <inertial>
+    <origin xyz="-0.011649938350470526 -0.011649938044416663 -0.0029692701223872214" rpy="0 0 0"/>
+    <mass value="0.004863692906073466"/>
     <inertia ixx="0.0" iyy="0.0" izz="1e-06" ixy="0.0" iyz="0.0" ixz="0.0"/>
   </inertial>
@@ -335,5 +337,5 @@
     <origin xyz="-0.09165 0.12535 0.1018" rpy="0 0 0"/>
     <geometry>
-      <mesh filename="package://test_bot/description/meshes/sim_caster_v7_1.stl" scale="0.001 0.001 0.001"/>
+      <mesh filename="package://test_bot/description/meshes/sim_caster_v8_1.stl" scale="0.001 0.001 0.001"/>
     </geometry>
     <material name="silver"/>
@@ -342,5 +344,5 @@
     <origin xyz="-0.09165 0.12535 0.1018" rpy="0 0 0"/>
     <geometry>
-      <mesh filename="package://test_bot/description/meshes/sim_caster_v7_1.stl" scale="0.001 0.001 0.001"/>
+      <mesh filename="package://test_bot/description/meshes/sim_caster_v8_1.stl" scale="0.001 0.001 0.001"/>
     </geometry>
   </collision>
@@ -363,4 +365,24 @@
     <geometry>
       <mesh filename="package://test_bot/description/meshes/sim_jet_v1_1.stl" scale="0.001 0.001 0.001"/>
+    </geometry>
+  </collision>
+</link>
+<link name="bola_v1_1">
+  <inertial>
+    <origin xyz="6.182422968015189e-08 6.195834001410105e-08 -1.7881401914721096e-10" rpy="0 0 0"/>
+    <mass value="0.004110250388446646"/>
+    <inertia ixx="0.0" iyy="0.0" izz="0.0" ixy="0.0" iyz="0.0" ixz="0.0"/>
+  </inertial>
+  <visual>
+    <origin xyz="-0.08 0.137 0.113" rpy="0 0 0"/>
+    <geometry>
+      <mesh filename="package://test_bot/description/meshes/bola_v1_1.stl" scale="0.001 0.001 0.001"/>
+    </geometry>
+    <material name="silver"/>
+  </visual>
+  <collision>
+    <origin xyz="-0.08 0.137 0.113" rpy="0 0 0"/>
+    <geometry>
+      <mesh filename="package://test_bot/description/meshes/bola_v1_1.stl" scale="0.001 0.001 0.001"/>
     </geometry>
   </collision>
@@ -446,5 +468,5 @@
   <origin xyz="0.00165 0.02165 -0.0358" rpy="0 0 0"/>
   <parent link="base_rueda_omni_v4_1"/>
-  <child link="sim_caster_v7_1"/>
+  <child link="sim_caster_v8_1"/>
 </joint>
 <joint name="Rigid 21" type="fixed">
@@ -453,9 +475,14 @@
   <child link="sim_jet_v1_1"/>
 </joint>
-<link name="esfera_deslizante_1">
+<joint name="Ball 22" type="fixed">
+  <origin xyz="-0.01165 -0.01165 -0.0112" rpy="0 0 0"/>
+  <parent link="sim_caster_v8_1"/>
+  <child link="bola_v1_1"/>
+</joint>
+<link name="esfera_deslizante">
   <inertial>
     <origin xyz="0 0 0" rpy="0 0 0"/>
-    <mass value="0.01"/>
-    <inertia ixx="1.2e-07" iyy="1.2e-07" izz="1.2e-07" ixy="0.0" iyz="0.0" ixz="0.0"/>
+    <mass value="0.004"/>
+    <inertia ixx="5e-08" iyy="5e-08" izz="5e-08" ixy="0.0" iyz="0.0" ixz="0.0"/>
   </inertial>
   <visual>
@@ -473,8 +500,33 @@
   </collision>
 </link>
-<joint name="Rigid_esfera_deslizante" type="fixed">
+<joint name="esfera_deslizante_joint" type="fixed">
   <origin xyz="0.08 -0.137 -0.116236" rpy="0 0 0"/>
   <parent link="body_link"/>
-  <child link="esfera_deslizante_1"/>
-</joint>
+  <child link="esfera_deslizante"/>
+</joint>
+<!-- ===================== ros2_control ===================== -->
+<!-- Replaces the old ROS 1 .trans transmissions. The gazebo_ros2_control
+     system plugin (see the .gazebo file) reads this block and the
+     controllers.yaml to bring up the controller_manager inside Gazebo. -->
+<ros2_control name="GazeboSystem" type="system">
+  <hardware>
+    <plugin>gazebo_ros2_control/GazeboSystem</plugin>
+  </hardware>
+  <joint name="left_wheel_joint">
+    <command_interface name="velocity">
+      <param name="min">-20.0</param>
+      <param name="max">20.0</param>
+    </command_interface>
+    <state_interface name="position"/>
+    <state_interface name="velocity"/>
+  </joint>
+  <joint name="right_wheel_joint">
+    <command_interface name="velocity">
+      <param name="min">-20.0</param>
+      <param name="max">20.0</param>
+    </command_interface>
+    <state_interface name="position"/>
+    <state_interface name="velocity"/>
+  </joint>
+</ros2_control>
 </robot>
